File: MCU/D11/starter_d11_rev2/Noise.kicad_sch (KiCad schematic)
At the start: 0 parts

Commit message: D11 schematics and PCB updates - printed prototype version
Parts:
- added C10, C9: 1µ, Capacitor_SMD:C_0805_2012Metric_Pad1.18x1.45mm_HandSolder, symbol Secoh:0805/C
- added C11: 0.01µ, Capacitor_SMD:C_0805_2012Metric_Pad1.18x1.45mm_HandSolder, symbol Secoh:0805/C
- added C12: 0.1µ, Capacitor_SMD:C_0805_2012Metric_Pad1.18x1.45mm_HandSolder, symbol Secoh:0805/C
- added C13, C7, C8: 2.2µ, Capacitor_SMD:C_0805_2012Metric_Pad1.18x1.45mm_HandSolder, symbol Secoh:0805/C
- added D2: 1N4007, Secoh:D_SOD-123F_hand_soldering, symbol Secoh:SOD-123/Diode
- added D3: SMF36A, Secoh:D_SOD-123F_hand_soldering, symbol Secoh:SOD-123/Zener
- added D4: SMF24A, Secoh:D_SOD-123F_hand_soldering, symbol Secoh:SOD-123/Zener
- added D5: MMBZ5222BLT1G, Package_TO_SOT_SMD:SOT-23_Handsoldering, symbol Secoh:SOD-123/Zener
- added J6: Conn_01x06_Pin, Connector_PinHeader_2.54mm:PinHeader_1x06_P2.54mm_Vertical, symbol Connector:Conn_01x06_Pin
- added L1: 100µ, Inductor_SMD:L_0805_2012Metric_Pad1.05x1.20mm_HandSolder, symbol ltspice:ind
- added R10, R15, R8: 10k, Resistor_SMD:R_0805_2012Metric_Pad1.20x1.40mm_HandSolder, symbol Secoh:0805/R
- added R11, R14, R17, R9: 100k, Resistor_SMD:R_0805_2012Metric_Pad1.20x1.40mm_HandSolder, symbol Secoh:0805/R
- added R12: 1Meg, Resistor_SMD:R_0805_2012Metric_Pad1.20x1.40mm_HandSolder, symbol Secoh:0805/R
- added R13: 47k, Resistor_SMD:R_0805_2012Metric_Pad1.20x1.40mm_HandSolder, symbol Secoh:0805/R
- added R16: 180, Resistor_SMD:R_0805_2012Metric_Pad1.20x1.40mm_HandSolder, symbol Secoh:0805/R
- added R6, R7: 33, Resistor_SMD:R_0805_2012Metric_Pad1.20x1.40mm_HandSolder, symbol Secoh:0805/R
- added SW2: Conn_01x03_Pin, Connector_PinHeader_2.54mm:PinHeader_1x03_P2.54mm_Vertical, symbol Connector:Conn_01x03_Pin
- added T1: 2N7002, Package_TO_SOT_SMD:SOT-23_Handsoldering, symbol Transistor_FET:2N7002
- added U3: MC74VHC1GT14, Package_TO_SOT_SMD:SOT-23-5_HandSoldering, symbol 74xGxx:74AHC1G14
- added U4: MAX4230, Package_TO_SOT_SMD:SOT-23-5_HandSoldering, symbol Secoh:OpAmp/MAX4230
- added U5: MIC1555, Package_TO_SOT_SMD:SOT-23-5_HandSoldering, symbol Secoh:Timer/MIC1555
Connections:
- new net: C13.1, R16.2, U5.4 (TRG), U5.5 (THR)
- new net: C11.1, D5.3 (K), R12.2, R13.2, U4.3 (-)
- new net: C10.1, R11.2, R8.1, R9.2
- new net: C9.1, D2.1 (K), D3.1 (K), R8.2
- new net: C11.2, D4.1 (K), R11.1
- new net: R17.1, SW2.2 (Pin_2), U3.2
- new net: R16.1, SW2.3 (Pin_3), U5.3 (OUT)
- new net: R14.1, R15.1, U4.1 (+)
- new net: T1.1 (G), U3.4
- new net: D2.2 (A), L1.2, T1.3 (D)
- new net: C7.1, R6.1, R7.2
- new net: C8.1, L1.1, R7.1
- new net 3V3-1: C12.1, J6.2 (Pin_2), R12.1, U4.5 (V+)
- new net 5V0-1: J6.1 (Pin_1), R17.2, R6.2, U3.5 (VCC), U5.1 (VCC)
- new net DRV: J6.4 (Pin_4), SW2.1 (Pin_1)
- new net GEN: J6.6 (Pin_6), R14.2, U4.4
- new net GND1: C10.2, C12.2, C13.2, C7.2, C8.2, C9.2, D3.2 (A), D4.2 (A), D5.1 (A), J6.3 (Pin_3), R10.1, R13.1, R15.2, T1.2 (S), U3.3 (GND), U4.2 (V-), U5.2 (GND)
- new net RDY: J6.5 (Pin_5), R10.2, R9.1
